Commit message: update urdf

File: urdf/mz04.urdf (robot description, URDF)
Before this commit: robot mz04, 9 links, 8 joints
Links:
- link flange_link: mass None -> 0.1
Joints:
- joint tool_joint: origin xyz=0.085 0 0.049 rpy=0 0 0 -> xyz=0.085 0 0.049 rpy=-3.141592 0 0

Commit message: エンドエフェクタの変更

File: urdf/mz04.urdf (robot description, URDF)
Before this commit: robot mz04, 9 links, 8 joints
Joints:
- joint tool_joint: origin xyz=0.085 0 0.049 rpy=-3.141592 0 0 -> xyz=0.095 0 0.049 rpy=-3.141592 0 0
